File: esphome-powermon.kicad_sch (KiCad schematic)
At the start: 22 parts, among them J1 Conn_01x15_Female, J11 Conn_01x15_Male, J12 Conn_01x15_Male, J13 Conn_01x04_Pin, J14 Conn_01x02_Pin, J15 Conn_01x04_Pin, J2 Conn_01x15_Female, J3 Conn_01x04_Pin, J4 Conn_01x02_Pin, J5 Conn_01x04_Pin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

Commit message: Replace burden resistor with TH footprint
Still for rev0.
Parts:
- R6: footprint Resistor_SMD:R_0603_1608Metric -> Resistor_THT:R_Axial_DIN0207_L6.3mm_D2.5mm_P7.62mm_Horizontal
Changed lines of the file:
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@@
       (effects (font (size 1.27 1.27)) (justify left))
     )
-    (property "Footprint" "Resistor_SMD:R_0603_1608Metric" (at 155.702 82.55 90)
+    (property "Footprint" "Resistor_THT:R_Axial_DIN0207_L6.3mm_D2.5mm_P7.62mm_Horizontal" (at 155.702 82.55 90)
       (effects (font (size 1.27 1.27)) hide)
     )

Commit message: Correct page markings
Parts:
- R6: LCSC C22962 -> (none)
Changed lines of the file:
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@@
   (title_block
     (title "ESPHome Power Monitor")
-    (date "2023-09-30")
-    (rev "2")
+    (date "2023-10-08")
+    (rev "0")
     (company "MichD")
   )
@@
       (effects (font (size 1.27 1.27)) hide)
     )
-    (property "LCSC" "C22962" (at 157.48 82.55 0)
-      (effects (font (size 1.27 1.27)) hide)
-    )
